Commit message: fix(bringup): re-calibrate RealSense bracket mount transforms
브라켓 위치가 잘못 잡혀 있어 재캘리브레이션:
- bracket_link joint origin xyz/rpy 재조정
- sensor_d435 카메라 origin xyz/rpy 재조정 (Y 부호 반전, rpy 중간값 보정)

File: src/m0609_rg2_bringup/urdf/realsense_bracket.urdf.xacro (robot description, xacro)
@@ -56,5 +56,5 @@
       xyz: 플랜지면이 tool0 원점에 오도록
     -->
-    <origin xyz="-0.002 -0.01 0.01" rpy="0 1.5708 -1.5708"/>
+    <origin xyz="-0.002 0.0 -0.01" rpy="0 -1.5708 1.5708"/>
   </joint>
   <!-- ───────────── RealSense D435 매크로 include ───────────── -->
@@ -64,5 +64,5 @@
   -->
   <xacro:sensor_d435 parent="bracket_link" name="camera" use_nominal_extrinsics="true">
-    <origin xyz="0 0.015 0.07" rpy="3.1416 0 1.5708"/>
+    <origin xyz="0.0 -0.015 0.05" rpy="3.1416 3.1416 1.5708"/>
   </xacro:sensor_d435>
 </robot>
