Commit message: feat(bringup): migrate to ROS 2 Jazzy with a single unified bringup
Jazzy breaks three assumptions the Humble launch relied on:

- controller_manager reads robot_description from a topic, not a parameter,
  so the old parameter-only wiring stalled at "Waiting for data on
  'robot_description' topic".
- Link and joint names changed (link1 -> link_1, joint1 -> joint_1).
- dsr_description2's xacro entry point has no tool0, unlike the static
  urdf/m0609.urdf the old URDF included.

One robot_description now covers both robot_state_publisher and
controller_manager: the combined URDF includes dsr_description2's xacro so
it carries <ros2_control> and the world link, and defines tool0 itself.
That also removes the separate static_transform_publisher.

bringup_camera.launch.py is folded into bringup.launch.py -- the two were
95% identical. The camera URDF is now always used (the bracket is bolted to
this robot) and the camera arg only controls the RealSense driver.

Adds rt_host, which the arm needs for the RT control channel on DRCF 3.0+;
without it an empty string reached the hardware parameters.

The virtual gripper now mirrors the real OnRobot driver: it publishes
/onrobot_joint_states with the driver's joint names and takes widths in
1/10 mm, so gripper_joint_state_publisher runs in both modes and everything
downstream of it is mode-independent. pick_place_demo.py drives a full
virtual pick and place cycle through the same /onrobot/sendCommand service.

File: src/m0609_rg2_bringup/urdf/m0609_with_rg2_camera.urdf.xacro (robot description, xacro)
@@ -1,11 +1,33 @@
 <?xml version="1.0"?>
+<!--
+  M0609 팔 + RG2 그리퍼 + RealSense 브라켓/D435 통합 URDF.
+  dsr_description2 의 정적 urdf/m0609.urdf 가 아니라 xacro/m0609.urdf.xacro 를 include 한다.
+  후자는 world 링크와 <ros2_control> 태그까지 만들어 주므로 이 한 장으로
+    - robot_state_publisher (RViz 표시 / TF)
+    - controller_manager (하드웨어 인터페이스 로드)
+  둘 다 커버된다. ROS2 Jazzy 의 controller_manager 는 robot_description 을 파라미터가 아니라
+  토픽에서 읽으므로, 두 노드가 같은 URDF 를 보게 하는 편이 갈라질 여지가 없다.
+  인자는 include 한 xacro/m0609.urdf.xacro 가 선언한 것을 그대로 쓴다:
+    xacro m0609_with_rg2_camera.urdf.xacro \
+      host:=127.0.0.1 port:=12345 mode:=virtual model:=m0609 update_rate:=100
+-->
 <robot xmlns:xacro="http://ros.org/wiki/xacro" name="m0609_rg2_camera">
-  <!-- M0609 URDF include -->
-  <xacro:include filename="$(find dsr_description2)/urdf/m0609.urdf"/>
-  <!-- RG2 macro include -->
+  <!-- 팔 (visual + world 링크 + ros2_control) -->
+  <xacro:include filename="$(find dsr_description2)/xacro/m0609.urdf.xacro"/>
+  <!-- RG2 매크로 -->
   <xacro:include filename="$(find m0609_rg2_bringup)/urdf/onrobot_rg2_model_macro.xacro"/>
-  <!-- RealSense 브라켓 + 카메라 include -->
+  <!-- RealSense 브라켓 + 카메라 -->
   <xacro:include filename="$(find m0609_rg2_bringup)/urdf/realsense_bracket.urdf.xacro"/>
-  <!-- RG2 그리퍼를 tool0에 부착 -->
+  <!-- 공구 장착 프레임.
+       정적 dsr_description2/urdf/m0609.urdf 에는 tool0 이 들어 있지만 xacro 쪽에는 없다.
+       그리퍼 / 브라켓이 모두 tool0 을 부모로 삼으므로 같은 변환으로 여기서 만든다
+       (urdf/m0609.urdf 의 joint_6-tool0 과 동일 origin). -->
+  <link name="tool0"/>
+  <joint name="joint_6-tool0" type="fixed">
+    <origin rpy="3.1415926535 -1.570796327 0" xyz="0 0 0"/>
+    <parent link="link_6"/>
+    <child link="tool0"/>
+  </joint>
+  <!-- RG2 그리퍼를 tool0 에 부착 (브라켓이 있어 오프셋 적용) -->
   <xacro:onrobot_rg2 prefix="rg2_" effector_base="tool0" has_bracket="true"/>
 </robot>
